Commit message: played around

File: haubentaucher_description/urdf/haubentaucher_base.urdf.xacro (robot description, xacro)
@@ -13,6 +13,6 @@
     <xacro:property name="prop_scale" value="0.0015" />
     <xacro:property name="mass" value="6.737"/>  <!-- [kg] --> <!-- changed values -->
-    <xacro:property name="body_width" value="0.47" /> <!-- [m] --> <!-- changed values -->
-    <xacro:property name="body_height" value="0.47" /> <!-- [m] --> <!-- changed values -->
+    <xacro:property name="body_width" value="0.51931" /> <!-- [m] --> <!-- updated 15.09.2023 -->
+    <xacro:property name="body_height" value="0.47305" /> <!-- [m] --> <!-- updated 15.09.2023 -->
     <xacro:property name="arm_length" value="0.354" /> <!-- [m] --> <!-- changed values -->
     <xacro:property name="rotor_x_offset" value="${arm_length*cos45}" /> <!-- [m] -->
@@ -35,5 +35,5 @@
     <xacro:property name="body_inertia">
         <!-- Iris values -->
-        <inertia ixx="0.02184" ixy="-0.001" ixz="-0.0131" iyy="0.2862" iyz="-0.0047" izz="0.1624" />  <!-- changed values -->
+        <inertia ixx="0.02953" ixy="0.0001" ixz="-0.0142" iyy="0.2303" iyz="0.0038" izz="0.1604" />  <!-- updated 15.09.2023 --> <!--inertia ixx="0.02953" ixy="0.0001" ixz="-0.0142" iyy="0.2303" iyz="0.0038" izz="0.1604" -->
     </xacro:property>
     <!-- inertia of a single rotor, assuming it is a cuboid. Height=3mm, width=15mm -->
@@ -41,10 +41,10 @@
         <xacro:box_inertia x="${radius_rotor}" y="0.015" z="0.003" mass="${mass_rotor*rotor_velocity_slowdown_sim}" />
     </xacro:property>
-    <xacro:property name="mesh_pos_x" value="-0.2175" /> <!-- [m] -->
-    <xacro:property name="mesh_pos_y" value="0.2175" /> <!-- [m] -->
-    <xacro:property name="mesh_pos_z" value="-0.05" /> <!-- [m] -->
-    <xacro:property name="mesh_ori_x" value="1.5707" /> <!-- [m] -->
-    <xacro:property name="mesh_ori_y" value="0.0" /> <!-- [m] -->
-    <xacro:property name="mesh_ori_z" value="0.0" /> <!-- [m] -->
+    <xacro:property name="robot_pos_x" value="0.0" /> <!-- [m] -->
+    <xacro:property name="robot_pos_y" value="0.0" /> <!-- [m] -->
+    <xacro:property name="robot_pos_z" value="0.0" /> <!-- [m] -->
+    <xacro:property name="robot_ori_x" value="0.0" /> <!-- [m] 1.5707 -->
+    <xacro:property name="robot_ori_y" value="0.0" /> <!-- [m] -->
+    <xacro:property name="robot_ori_z" value="0.0" /> <!-- [m] -->
     <xacro:property name="mesh_aerprop_pos_x" value="0.1905" /> <!-- [m] -->
     <xacro:property name="mesh_aerprop_pos_y" value="-0.0205" /> <!-- [m] -->
@@ -63,5 +63,5 @@
          mesh_file="${mesh_file}"
          mesh_scale="${mesh_scale}">
-         <origin xyz="${mesh_pos_x} ${mesh_pos_y} ${mesh_pos_z}" rpy="${mesh_ori_x} ${mesh_ori_y} ${mesh_ori_z}"/>
+         <origin xyz="${robot_pos_x} ${robot_pos_y} ${robot_pos_z}" rpy="${robot_ori_x} ${robot_ori_y} ${robot_ori_z}"/>
          <xacro:insert_block name="body_inertia" />
     </xacro:multirotor_base_macro>

File: haubentaucher_description/urdf/multirotor_base.urdf.xacro (robot description, xacro)
@@ -54,4 +54,5 @@
           <!--box size="${body_width} ${body_width} ${body_height}"/--> <!-- [m] [m] [m] -->
         </geometry>
+        <origin xyz="-${body_width/2 + 0.015} -${body_width/2 + 0.015} 0" rpy="0 0 0"/> <!-- 0.015 found out by iteration -->
       </visual>
       <collision>
@@ -61,4 +62,5 @@
           <box size="${body_width} ${body_width} ${body_height}"/> <!-- [m] [m] [m] -->
         </geometry>
+        <origin xyz="0 0 ${body_height/2 + 0.015}" rpy="0 0 0"/> <!-- 0.015 found out by iteration -->
       </collision>
     </link>

Commit message: update

File: haubentaucher_description/urdf/haubentaucher_base.urdf.xacro (robot description, xacro)
@@ -7,11 +7,11 @@
     <!-- Body Properties -->
     <xacro:property name="rotor_velocity_slowdown_sim" value="10" />
-    <xacro:property name="mesh_file" value="haubentaucher_description/meshes/Haubentaucher.STL" /> <!-- changed (change name someday) -->
+    <xacro:property name="mesh_file" value="$(find haubentaucher_description)/meshes/untitled.stl" /> <!-- changed (change name someday) -->
     <xacro:property name="rotor_1_mesh_file" value="haubentaucher_description/meshes/aerial_propeller_1.dae" />
     <xacro:property name="rotor_2_mesh_file" value="haubentaucher_description/meshes/aerial_propeller_2.dae" />
-    <xacro:property name="mesh_scale" value="0.001" />
+    <xacro:property name="mesh_scale" value="1" />
     <xacro:property name="prop_scale" value="0.0015" />
     <xacro:property name="mass" value="6.737"/>  <!-- [kg] --> <!-- changed values -->
-    <xacro:property name="body_width" value="0.51931" /> <!-- [m] --> <!-- updated 15.09.2023 -->
+    <xacro:property name="body_width" value="0.21931" /> <!-- [m] --> <!-- updated 15.09.2023 -->
     <xacro:property name="body_height" value="0.47305" /> <!-- [m] --> <!-- updated 15.09.2023 -->
     <xacro:property name="arm_length" value="0.354" /> <!-- [m] --> <!-- changed values -->
@@ -19,4 +19,5 @@
     <xacro:property name="rotor_y_offset" value="${arm_length*sin45}" /> <!-- [m] -->
     <xacro:property name="rotor_offset_top" value="0.035" /> <!-- [m] -->
+    <xacro:property name="use_mesh_file" value="true" />
     <!-- Rotor constants -->
     <xacro:property name="mass_rotor" value="0.005" /> <!-- [kg] -->
@@ -53,6 +54,7 @@
     <xacro:property name="mesh_aerprop_ori_y" value="0.0" /> <!-- [m] -->
     <xacro:property name="mesh_aerprop_ori_z" value="1.5707" /> <!-- [m] -->
-    <!-- Included URDF Files -->
-    <xacro:include filename="$(find haubentaucher_description)/urdf/multirotor_base.urdf.xacro" />
+    <!-- Included URDF Files
+    <xacro:include filename="$(find haubentaucher_description)/urdf/multirotor_base.urdf.xacro" /> -->
+    <xacro:include filename="$(find haubentaucher_description)/urdf/haubentaucher_multirotor_base.xacro" />
     <!-- Instantiate multirotor_base_macro once -->
     <xacro:multirotor_base_macro
@@ -61,90 +63,95 @@
          body_width="${body_width}"
          body_height="${body_height}"
+         use_mesh_file="${use_mesh_file}"
          mesh_file="${mesh_file}"
-         mesh_scale="${mesh_scale}">
-         <origin xyz="${robot_pos_x} ${robot_pos_y} ${robot_pos_z}" rpy="${robot_ori_x} ${robot_ori_y} ${robot_ori_z}"/>
+         mesh_scale="${mesh_scale}"
+         >
          <xacro:insert_block name="body_inertia" />
     </xacro:multirotor_base_macro>
     <!-- Instantiate rotors -->
-    <xacro:vertical_rotor
-        robot_namespace="${namespace}"
-        suffix="front_right"
-        direction="ccw"
-        motor_constant="${motor_constant}"
-        moment_constant="${moment_constant}"
-        parent="${namespace}/base_link"
-        mass_rotor="${mass_rotor}"
-        radius_rotor="${radius_rotor}"
-        time_constant_up="${time_constant_up}"
-        time_constant_down="${time_constant_down}"
-        max_rot_velocity="${max_rot_velocity}"
-        motor_number="0"
-        rotor_drag_coefficient="${rotor_drag_coefficient}"
-        rolling_moment_coefficient="${rolling_moment_coefficient}"
-        color="Blue"
-        prop_scale="${prop_scale}">
-        <origin xyz="${arm_length} -${arm_length} ${rotor_offset_top}" rpy="0 0 0" />
-        <xacro:insert_block name="rotor_inertia" />
-    </xacro:vertical_rotor>
-    <xacro:vertical_rotor
-        robot_namespace="${namespace}"
-        suffix="back_left"
-        direction="ccw"
-        motor_constant="${motor_constant}"
-        moment_constant="${moment_constant}"
-        parent="${namespace}/base_link"
-        mass_rotor="${mass_rotor}"
-        radius_rotor="${radius_rotor}"
-        time_constant_up="${time_constant_up}"
-        time_constant_down="${time_constant_down}"
-        max_rot_velocity="${max_rot_velocity}"
-        motor_number="1"
-        rotor_drag_coefficient="${rotor_drag_coefficient}"
-        rolling_moment_coefficient="${rolling_moment_coefficient}"
-        color="Blue"
-        prop_scale="${prop_scale}">
-        <origin xyz="-${arm_length} ${arm_length} ${rotor_offset_top}" rpy="0 0 0" />
-        <xacro:insert_block name="rotor_inertia" />
-    </xacro:vertical_rotor>
-    <xacro:vertical_rotor
-        robot_namespace="${namespace}"
-        suffix="front_left"
-        direction="cw"
-        motor_constant="${motor_constant}"
-        moment_constant="${moment_constant}"
-        parent="${namespace}/base_link"
-        mass_rotor="${mass_rotor}"
-        radius_rotor="${radius_rotor}"
-        time_constant_up="${time_constant_up}"
-        time_constant_down="${time_constant_down}"
-        max_rot_velocity="${max_rot_velocity}"
-        motor_number="2"
-        rotor_drag_coefficient="${rotor_drag_coefficient}"
-        rolling_moment_coefficient="${rolling_moment_coefficient}"
-        color="Blue"
-        prop_scale="${prop_scale}">
-        <origin xyz="${arm_length} ${arm_length} ${rotor_offset_top}" rpy="0 0 0" />
-        <xacro:insert_block name="rotor_inertia" />
-    </xacro:vertical_rotor>
-    <xacro:vertical_rotor
-        robot_namespace="${namespace}"
-        suffix="back_right"
-        direction="cw"
-        motor_constant="${motor_constant}"
-        moment_constant="${moment_constant}"
-        parent="${namespace}/base_link"
-        mass_rotor="${mass_rotor}"
-        radius_rotor="${radius_rotor}"
-        time_constant_up="${time_constant_up}"
-        time_constant_down="${time_constant_down}"
-        max_rot_velocity="${max_rot_velocity}"
-        motor_number="3"
-        rotor_drag_coefficient="${rotor_drag_coefficient}"
-        rolling_moment_coefficient="${rolling_moment_coefficient}"
-        color="Blue"
-        prop_scale="${prop_scale}">
-        <origin xyz="-${arm_length} -${arm_length} ${rotor_offset_top}" rpy="0 0 0" />
-        <xacro:insert_block name="rotor_inertia" />
-    </xacro:vertical_rotor>
+  <xacro:vertical_rotor
+    robot_namespace="${namespace}"
+    suffix="front"
+    direction="cw"
+    motor_constant="${motor_constant}"
+    moment_constant="${moment_constant}"
+    parent="${namespace}/base_link"
+    mass_rotor="${mass_rotor}"
+    radius_rotor="${radius_rotor}"
+    time_constant_up="${time_constant_up}"
+    time_constant_down="${time_constant_down}"
+    max_rot_velocity="${max_rot_velocity}"
+    motor_number="0"
+    rotor_drag_coefficient="${rotor_drag_coefficient}"
+    rolling_moment_coefficient="${rolling_moment_coefficient}"
+    color="Red"
+    use_own_mesh="false"
+    mesh="">
+    <origin xyz="${arm_length} 0 ${rotor_offset_top}" rpy="0 0 0" />
+    <xacro:insert_block name="rotor_inertia" />
+  </xacro:vertical_rotor>
+  <xacro:vertical_rotor
+    robot_namespace="${namespace}"
+    suffix="left"
+    direction="ccw"
+    motor_constant="${motor_constant}"
+    moment_constant="${moment_constant}"
+    parent="${namespace}/base_link"
+    mass_rotor="${mass_rotor}"
+    radius_rotor="${radius_rotor}"
+    time_constant_up="${time_constant_up}"
+    time_constant_down="${time_constant_down}"
+    max_rot_velocity="${max_rot_velocity}"
+    motor_number="1"
+    rotor_drag_coefficient="${rotor_drag_coefficient}"
+    rolling_moment_coefficient="${rolling_moment_coefficient}"
+    color="Blue"
+    use_own_mesh="false"
+    mesh="">
+    <origin xyz="0 ${arm_length} ${rotor_offset_top}" rpy="0 0 0" />
+    <xacro:insert_block name="rotor_inertia" />
+  </xacro:vertical_rotor>
+  <xacro:vertical_rotor
+    robot_namespace="${namespace}"
+    suffix="back"
+    direction="cw"
+    motor_constant="${motor_constant}"
+    moment_constant="${moment_constant}"
+    parent="${namespace}/base_link"
+    mass_rotor="${mass_rotor}"
+    radius_rotor="${radius_rotor}"
+    time_constant_up="${time_constant_up}"
+    time_constant_down="${time_constant_down}"
+    max_rot_velocity="${max_rot_velocity}"
+    motor_number="2"
+    rotor_drag_coefficient="${rotor_drag_coefficient}"
+    rolling_moment_coefficient="${rolling_moment_coefficient}"
+    color="Blue"
+    use_own_mesh="false"
+    mesh="">
+    <origin xyz="-${arm_length} 0 ${rotor_offset_top}" rpy="0 0 0" />
+    <xacro:insert_block name="rotor_inertia" />
+  </xacro:vertical_rotor>
+  <xacro:vertical_rotor
+    robot_namespace="${namespace}"
+    suffix="right"
+    direction="ccw"
+    motor_constant="${motor_constant}"
+    moment_constant="${moment_constant}"
+    parent="${namespace}/base_link"
+    mass_rotor="${mass_rotor}"
+    radius_rotor="${radius_rotor}"
+    time_constant_up="${time_constant_up}"
+    time_constant_down="${time_constant_down}"
+    max_rot_velocity="${max_rot_velocity}"
+    motor_number="3"
+    rotor_drag_coefficient="${rotor_drag_coefficient}"
+    rolling_moment_coefficient="${rolling_moment_coefficient}"
+    color="Blue"
+    use_own_mesh="false"
+    mesh="">
+    <origin xyz="0 -${arm_length} ${rotor_offset_top}" rpy="0 0 0" />
+    <xacro:insert_block name="rotor_inertia" />
+  </xacro:vertical_rotor>
     <gazebo reference="$(arg namespace)/base_link">
         <dampingFactor>0.001</dampingFactor>

Commit message: update

File: haubentaucher_description/urdf/haubentaucher_base.urdf.xacro (robot description, xacro)
@@ -15,8 +15,8 @@
     <xacro:property name="body_width" value="0.21931" /> <!-- [m] --> <!-- updated 15.09.2023 -->
     <xacro:property name="body_height" value="0.47305" /> <!-- [m] --> <!-- updated 15.09.2023 -->
-    <xacro:property name="arm_length" value="0.354" /> <!-- [m] --> <!-- changed values -->
+    <xacro:property name="arm_length" value="0.316" /> <!-- [m] --> <!-- changed values -->
     <xacro:property name="rotor_x_offset" value="${arm_length*cos45}" /> <!-- [m] -->
     <xacro:property name="rotor_y_offset" value="${arm_length*sin45}" /> <!-- [m] -->
-    <xacro:property name="rotor_offset_top" value="0.035" /> <!-- [m] -->
+    <xacro:property name="rotor_offset_top" value="0.157" /> <!-- [m] -->
     <xacro:property name="use_mesh_file" value="true" />
     <!-- Rotor constants -->
@@ -42,16 +42,4 @@
         <xacro:box_inertia x="${radius_rotor}" y="0.015" z="0.003" mass="${mass_rotor*rotor_velocity_slowdown_sim}" />
     </xacro:property>
-    <xacro:property name="robot_pos_x" value="0.0" /> <!-- [m] -->
-    <xacro:property name="robot_pos_y" value="0.0" /> <!-- [m] -->
-    <xacro:property name="robot_pos_z" value="0.0" /> <!-- [m] -->
-    <xacro:property name="robot_ori_x" value="0.0" /> <!-- [m] 1.5707 -->
-    <xacro:property name="robot_ori_y" value="0.0" /> <!-- [m] -->
-    <xacro:property name="robot_ori_z" value="0.0" /> <!-- [m] -->
-    <xacro:property name="mesh_aerprop_pos_x" value="0.1905" /> <!-- [m] -->
-    <xacro:property name="mesh_aerprop_pos_y" value="-0.0205" /> <!-- [m] -->
-    <xacro:property name="mesh_aerprop_pos_z" value="0.01" /> <!-- [m] -->
-    <xacro:property name="mesh_aerprop_ori_x" value="-1.5707" /> <!-- [m] -->
-    <xacro:property name="mesh_aerprop_ori_y" value="0.0" /> <!-- [m] -->
-    <xacro:property name="mesh_aerprop_ori_z" value="1.5707" /> <!-- [m] -->
     <!-- Included URDF Files
     <xacro:include filename="$(find haubentaucher_description)/urdf/multirotor_base.urdf.xacro" /> -->
@@ -88,5 +76,5 @@
     use_own_mesh="false"
     mesh="">
-    <origin xyz="${arm_length} 0 ${rotor_offset_top}" rpy="0 0 0" />
+    <origin xyz="${rotor_x_offset} ${rotor_y_offset} ${rotor_offset_top}" rpy="0 0 0" />
     <xacro:insert_block name="rotor_inertia" />
   </xacro:vertical_rotor>
@@ -109,5 +97,5 @@
     use_own_mesh="false"
     mesh="">
-    <origin xyz="0 ${arm_length} ${rotor_offset_top}" rpy="0 0 0" />
+    <origin xyz="${rotor_x_offset} -${rotor_y_offset} ${rotor_offset_top}" rpy="0 0 0" />
     <xacro:insert_block name="rotor_inertia" />
   </xacro:vertical_rotor>
@@ -130,5 +118,5 @@
     use_own_mesh="false"
     mesh="">
-    <origin xyz="-${arm_length} 0 ${rotor_offset_top}" rpy="0 0 0" />
+    <origin xyz="-${rotor_x_offset} ${rotor_y_offset} ${rotor_offset_top}" rpy="0 0 0" />
     <xacro:insert_block name="rotor_inertia" />
   </xacro:vertical_rotor>
@@ -151,5 +139,5 @@
     use_own_mesh="false"
     mesh="">
-    <origin xyz="0 -${arm_length} ${rotor_offset_top}" rpy="0 0 0" />
+    <origin xyz="-${rotor_x_offset} -${rotor_y_offset} ${rotor_offset_top}" rpy="0 0 0" />
     <xacro:insert_block name="rotor_inertia" />
   </xacro:vertical_rotor>

Commit message: update

File: haubentaucher_description/urdf/haubentaucher_base.urdf.xacro (robot description, xacro)
@@ -18,5 +18,5 @@
     <xacro:property name="rotor_x_offset" value="${arm_length*cos45}" /> <!-- [m] -->
     <xacro:property name="rotor_y_offset" value="${arm_length*sin45}" /> <!-- [m] -->
-    <xacro:property name="rotor_offset_top" value="0.157" /> <!-- [m] -->
+    <xacro:property name="rotor_offset_top" value="0.165" /> <!-- [m] --> <!-- find out with iteration -->
     <xacro:property name="use_mesh_file" value="true" />
     <!-- Rotor constants -->
@@ -76,5 +76,5 @@
     use_own_mesh="false"
     mesh="">
-    <origin xyz="${rotor_x_offset} ${rotor_y_offset} ${rotor_offset_top}" rpy="0 0 0" />
+    <origin xyz="${rotor_x_offset} ${rotor_y_offset} ${rotor_offset_top}" rpy="0 0 0" /> <!-- look at the definition above to understand how the position is defined -->
     <xacro:insert_block name="rotor_inertia" />
   </xacro:vertical_rotor>

Commit message: collision

File: haubentaucher_description/urdf/haubentaucher_base.urdf.xacro (robot description, xacro)
@@ -7,5 +7,5 @@
     <!-- Body Properties -->
     <xacro:property name="rotor_velocity_slowdown_sim" value="10" />
-    <xacro:property name="mesh_file" value="$(find haubentaucher_description)/meshes/untitled.stl" /> <!-- changed (change name someday) -->
+    <xacro:property name="mesh_file" value="$(find haubentaucher_description)/meshes/haubentaucher_centered.stl" /> <!-- import mesh file -->
     <xacro:property name="rotor_1_mesh_file" value="haubentaucher_description/meshes/aerial_propeller_1.dae" />
     <xacro:property name="rotor_2_mesh_file" value="haubentaucher_description/meshes/aerial_propeller_2.dae" />
@@ -13,5 +13,5 @@
     <xacro:property name="prop_scale" value="0.0015" />
     <xacro:property name="mass" value="6.737"/>  <!-- [kg] --> <!-- changed values -->
-    <xacro:property name="body_width" value="0.21931" /> <!-- [m] --> <!-- updated 15.09.2023 -->
+    <xacro:property name="body_width" value="0.15" /> <!-- [m] --> <!-- updated 15.09.2023 -->
     <xacro:property name="body_height" value="0.47305" /> <!-- [m] --> <!-- updated 15.09.2023 -->
     <xacro:property name="arm_length" value="0.316" /> <!-- [m] --> <!-- changed values -->

Commit message: inertia comment

File: haubentaucher_description/urdf/haubentaucher_base.urdf.xacro (robot description, xacro)
@@ -36,5 +36,5 @@
     <xacro:property name="body_inertia">
         <!-- Iris values -->
-        <inertia ixx="0.02953" ixy="0.0001" ixz="-0.0142" iyy="0.2303" iyz="0.0038" izz="0.1604" />  <!-- updated 15.09.2023 --> <!--inertia ixx="0.02953" ixy="0.0001" ixz="-0.0142" iyy="0.2303" iyz="0.0038" izz="0.1604" -->
+        <inertia ixx="0.02953" ixy="0.0001" ixz="-0.0142" iyy="0.2303" iyz="0.0038" izz="0.1604" />  <!-- updated 15.09.2023 -->
     </xacro:property>
     <!-- inertia of a single rotor, assuming it is a cuboid. Height=3mm, width=15mm -->

Commit message: inertia update

File: haubentaucher_description/urdf/haubentaucher_base.urdf.xacro (robot description, xacro)
@@ -7,13 +7,13 @@
     <!-- Body Properties -->
     <xacro:property name="rotor_velocity_slowdown_sim" value="10" />
-    <xacro:property name="mesh_file" value="$(find haubentaucher_description)/meshes/haubentaucher_centered.stl" /> <!-- import mesh file -->
+    <xacro:property name="mesh_file" value="$(find haubentaucher_description)/meshes/haubentaucher_centered.stl" /> <!-- import mesh file haubentaucher_centered.stl-->
     <xacro:property name="rotor_1_mesh_file" value="haubentaucher_description/meshes/aerial_propeller_1.dae" />
     <xacro:property name="rotor_2_mesh_file" value="haubentaucher_description/meshes/aerial_propeller_2.dae" />
-    <xacro:property name="mesh_scale" value="1" />
+    <xacro:property name="mesh_scale" value="1" /> <!--1-->
     <xacro:property name="prop_scale" value="0.0015" />
     <xacro:property name="mass" value="6.737"/>  <!-- [kg] --> <!-- changed values -->
     <xacro:property name="body_width" value="0.15" /> <!-- [m] --> <!-- updated 15.09.2023 -->
     <xacro:property name="body_height" value="0.47305" /> <!-- [m] --> <!-- updated 15.09.2023 -->
-    <xacro:property name="arm_length" value="0.316" /> <!-- [m] --> <!-- changed values -->
+    <xacro:property name="arm_length" value="0.316" /> <!-- [m] --> <!-- changed values 0.316-->
     <xacro:property name="rotor_x_offset" value="${arm_length*cos45}" /> <!-- [m] -->
     <xacro:property name="rotor_y_offset" value="${arm_length*sin45}" /> <!-- [m] -->
@@ -36,5 +36,5 @@
     <xacro:property name="body_inertia">
         <!-- Iris values -->
-        <inertia ixx="0.02953" ixy="0.0001" ixz="-0.0142" iyy="0.2303" iyz="0.0038" izz="0.1604" />  <!-- updated 15.09.2023 -->
+        <inertia ixx="0.2284" ixy="0.0003" ixz="-0.0091" iyy="0.1633" iyz="0.0011" izz="0.1599" />  <!-- updated 03.10.2023 --> <!-- 15.09.2023 ixx="0.02953" ixy="0.0001" ixz="-0.0142" iyy="0.2303"  iyz="0.0038" izz="0.1604"-->
     </xacro:property>
     <!-- inertia of a single rotor, assuming it is a cuboid. Height=3mm, width=15mm -->
